File: eagle/LightControl5C.brd (EAGLE design)
At the start: 43.2 x 26.7 mm, 36 parts, among them IC1 LV3842XF, IC2 PIC12F675, IC3 7805, U1 ULN2003D, X1 Footprint, X10 Footprint, X11 Footprint, X2 Footprint, X3 FLE-103-01, X4 Footprint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

Commit message: [eagle] change inductor
-> increase min. inductor size to allow lower currents
Parts:
- L1: value 33µ -> 150µ
Changed lines of the file:
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@@
 <attribute name="NAME" x="19.685" y="6.985" size="0.8128" layer="25" font="vector" ratio="15" rot="R90"/>
 </element>
-<element name="L1" library="omcInductor" package="PISM" value="33µ" x="13.335" y="8.89" smashed="yes" rot="R270">
-<attribute name="DIST#REICHELT#" value="L-PISM 33µ" x="13.335" y="8.89" size="1.778" layer="27" rot="R270" display="off"/>
-<attribute name="VENDOR#" value="Fastron,PISM-330X-04" x="13.335" y="8.89" size="1.778" layer="27" rot="R270" display="off"/>
+<element name="L1" library="omcInductor" package="PISM" value="150µ" x="13.335" y="8.89" smashed="yes" rot="R270">
+<attribute name="DIST#REICHELT#" value="L-PISM 150µ" x="13.335" y="8.89" size="1.778" layer="27" rot="R270" display="off"/>
+<attribute name="VENDOR#" value="Fastron,PISM-151X-04" x="13.335" y="8.89" size="1.778" layer="27" rot="R270" display="off"/>
 <attribute name="DIST#DIGIKEY#" value="" x="13.335" y="8.89" size="1.778" layer="27" rot="R270" display="off"/>
 <attribute name="DIST#CONRAD#" value="" x="13.335" y="8.89" size="1.778" layer="27" rot="R270" display="off"/>
